Commit message: add odom

File: xacro/diff_wheel_robo3.xacro (robot description, xacro)
@@ -2,8 +2,8 @@
 <robot name="dtw_robot" xmlns:xacro="http://ros.org/wiki/xacro">
   <material name="gray">
-    <color rgba="0.5 0.5 0.5 2.5"/>
+    <color rgba="0.5 0.5 0.5 1.0"/>
   </material>
   <material name="red">
-    <color rgba="1.0 0.0 0.0 2.5"/>
+    <color rgba="1.0 0.0 0.0 1.0"/>
   </material>
   <xacro:macro name="wheel_macro" params="parent prefix xyz">
@@ -13,11 +13,11 @@
       <child  link="${prefix}_link"/>
       <axis xyz="0 0 1" />
-      <limit velocity="12.0" effort="0.4"/>
+      <limit velocity="12.0" effort="0.4" />
       <dynamics damping="0.1"/>
     </joint>
-    <transmission name="${prefix}_trans" type="SImpleTransmission">
+    <transmission name="${prefix}_trans" type="SimpleTransmission">
       <type>transmission_interface/SimpleTransmission</type>
       <actuator name="${prefix}_motor">
-        <mechanismReduction>1</mechanismReduction>
+        <mechanicalReduction>1</mechanicalReduction>
       </actuator>
       <joint name="${prefix}_joint">
@@ -32,5 +32,4 @@
       </inertial>
       <visual>
-        <origin xyz="0 0 0" rpy="0 0 0"/>
         <geometry>
           <cylinder radius="0.05" length="0.02" />
@@ -39,5 +38,4 @@
       </visual>
       <collision>
-        <origin xyz="0 0 0" rpy="0 0 0"/>
         <geometry>
           <cylinder radius="0.05" length="0.02"/>
@@ -50,5 +48,5 @@
       <mu2 value="2.5"/>
       <kp value="50000"/>
-      <kp value="10"/>
+      <kd value="10"/>
     </gazebo>
   </xacro:macro>
@@ -75,5 +73,5 @@
       <origin xyz="0 0 0" rpy="0 0 0"/>
       <geometry>
-        <box size="0.24 0.178 0.06"/>
+        <box size="0.24 0.17 0.06"/>
       </geometry>
     </collision>
@@ -112,8 +110,16 @@
   <gazebo>
     <plugin name="gazebo_ros_control" filename="libgazebo_ros_control.so">
-      <robotNameSpace>/dtw_robot</robotNameSpace>
+      <robotNamespace>/dtw_robot</robotNamespace>
       <robotSimType>gazebo_ros_control/DefaultRobotHWSim</robotSimType>
       <legacyModeNS>true</legacyModeNS>
     </plugin>
   </gazebo>
+    <gazebo>
+    <plugin name="ground_truth" filename="libgazebo_ros_p3d.so">
+      <frameName>world</frameName>
+      <bodyName>base_link</bodyName>
+      <topicName>/tracker</topicName>
+      <updateRate>10.0</updateRate>
+    </plugin>
+  </gazebo>
 </robot>
